File: Columba2/multiplex2.sch (EAGLE design)
At the start: 21 parts, among them U1 MAX4617CUE+T

Commit message: Add files via upload
Parts:
- removed R1, R2, R3, R4: 10k, SparkFun-Resistors:10KOHM-0603-1/10W-1%
- added C1: 10uf, OPL_Capacitor:CERAMIC-10UF-25V-10%-X5R(1206)
- added JP3: (no value), adafruit:PINHD-1X1
- R5: value 100k -> 10k
Connections:
- removed net N$5: Q3.G, R3.2
- removed net N$6: Q5.G, R1.2
- removed net N$7: Q4.G, R2.2
- removed net N$9: Q1.G, R4.2
- new net X: JL1.P$5, U1.X
- net 5V: now also C1.1
- net GND: now also C1.2
- net N$8: now also JP3.1
- net PX_EN: no longer JL1.P$5
- net SV0: now also Q5.G; no longer R1.1
- net SV1: now also Q4.G; no longer R2.1
- net SV2: now also Q3.G; no longer R3.1
- net SV3: now also Q1.G; no longer R4.1

Commit message: Add files via upload
Parts:
- removed JP1, JP2: (no value), adafruit:PINHD-1X1
- added J1: LIGHT, SparkFun-Connectors:CONN_02
- JP3: value (none) -> extra
Connections:
- net 5V: now also J1.2; no longer JP1.1
- net LIGHT_S: now also J1.1; no longer JP2.1
- net PX_EN: now also JL1.P$3
- net SV0: now also JL1.P$2; no longer JL1.P$12
- net SV1: now also JL1.P$4; no longer JL1.P$10
Changed lines of the file:
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@@
 <part name="Q4" library="adafruit" deviceset="MOSFET-N" device="REFLOW"/>
 <part name="Q5" library="adafruit" deviceset="MOSFET-N" device="REFLOW"/>
-<part name="JP1" library="adafruit" library_urn="urn:adsk.eagle:library:420" deviceset="PINHD-1X1" device="" package3d_urn="urn:adsk.eagle:package:6240654/1"/>
-<part name="JP2" library="adafruit" library_urn="urn:adsk.eagle:library:420" deviceset="PINHD-1X1" device="" package3d_urn="urn:adsk.eagle:package:6240654/1"/>
 <part name="R5" library="SparkFun-Resistors" library_urn="urn:adsk.eagle:library:532" deviceset="100KOHM" device="-0603-1/10W-1%" package3d_urn="urn:adsk.eagle:package:39650/1" value="10k"/>
 <part name="GND2" library="custom" deviceset="GND" device=""/>
-<part name="GND1" library="custom" deviceset="GND" device=""/>
 <part name="C1" library="OPL_Capacitor" library_urn="urn:adsk.eagle:library:8004261" deviceset="CERAMIC-10UF-25V-10%-X5R(1206)" device="" package3d_urn="urn:adsk.eagle:package:8004280/1" value="10uf"/>
-<part name="JP3" library="adafruit" library_urn="urn:adsk.eagle:library:420" deviceset="PINHD-1X1" device="" package3d_urn="urn:adsk.eagle:package:6240654/1"/>
+<part name="JP3" library="adafruit" library_urn="urn:adsk.eagle:library:420" deviceset="PINHD-1X1" device="" package3d_urn="urn:adsk.eagle:package:6240654/1" value="extra"/>
+<part name="J1" library="SparkFun-Connectors" library_urn="urn:adsk.eagle:library:513" deviceset="CONN_02" device="" package3d_urn="urn:adsk.eagle:package:38039/1" value="LIGHT"/>
 </parts>
 <sheets>
@@
 <instance part="Q4" gate="G$1" x="30.48" y="-53.34" rot="MR270"/>
 <instance part="Q5" gate="G$1" x="30.48" y="-66.04" rot="MR270"/>
-<instance part="JP1" gate="G$1" x="106.68" y="-33.02"/>
-<instance part="JP2" gate="G$1" x="116.84" y="-33.02"/>
 <instance part="R5" gate="G$1" x="114.3" y="-45.72" rot="R270"/>
 <instance part="GND2" gate="G$1" x="114.3" y="-66.04"/>
-<instance part="GND1" gate="G$1" x="35.56" y="-81.28"/>
 <instance part="C1" gate="G$1" x="58.42" y="25.4" rot="R180"/>
 <instance part="JP3" gate="G$1" x="132.08" y="-10.16"/>
+<instance part="J1" gate="G$1" x="111.76" y="-25.4" rot="R90"/>
 </instances>
 <busses>
@@
 </segment>
 <segment>
-<pinref part="JP1" gate="G$1" pin="1"/>
-<wire x1="104.14" y1="-33.02" x2="104.14" y2="-43.18" width="0.1524" layer="91"/>
 <label x="106.68" y="-43.18" size="1.778" layer="95" rot="R90"/>
+<wire x1="104.14" y1="-43.18" x2="104.14" y2="-17.78" width="0.1524" layer="91"/>
+<pinref part="J1" gate="G$1" pin="2"/>
+<wire x1="104.14" y1="-17.78" x2="109.22" y2="-17.78" width="0.1524" layer="91"/>
 </segment>
 </net>
@@
 <label x="205.74" y="-86.36" size="1.778" layer="95" rot="R180" xref="yes"/>
 </segment>
+<segment>
+<pinref part="JL1" gate="G$1" pin="P$3"/>
+<wire x1="77.47" y1="53.34" x2="83.82" y2="53.34" width="0.1524" layer="91"/>
+<label x="83.82" y="53.34" size="1.778" layer="95"/>
+</segment>
 </net>
 <net name="LIGHT_S" class="0">
 <segment>
 <label x="114.3" y="-5.08" size="1.778" layer="95"/>
-<pinref part="JP2" gate="G$1" pin="1"/>
 <pinref part="R5" gate="G$1" pin="1"/>
-<wire x1="114.3" y1="-40.64" x2="114.3" y2="-33.02" width="0.1524" layer="91"/>
+<wire x1="114.3" y1="-40.64" x2="114.3" y2="-17.78" width="0.1524" layer="91"/>
 <pinref part="U1" gate="G$1" pin="X6"/>
 <wire x1="104.14" y1="-5.08" x2="121.92" y2="-5.08" width="0.1524" layer="91"/>
-<wire x1="121.92" y1="-5.08" x2="121.92" y2="-33.02" width="0.1524" layer="91"/>
-<wire x1="121.92" y1="-33.02" x2="114.3" y2="-33.02" width="0.1524" layer="91"/>
-<junction x="114.3" y="-33.02"/>
+<wire x1="121.92" y1="-5.08" x2="121.92" y2="-17.78" width="0.1524" layer="91"/>
+<wire x1="121.92" y1="-17.78" x2="114.3" y2="-17.78" width="0.1524" layer="91"/>
+<pinref part="J1" gate="G$1" pin="1"/>
+<wire x1="114.3" y1="-17.78" x2="111.76" y2="-17.78" width="0.1524" layer="91"/>
+<junction x="114.3" y="-17.78"/>
 </segment>
 </net>
@@
 <net name="SV0" class="0">
 <segment>
-<pinref part="JL1" gate="G$1" pin="P$12"/>
-<wire x1="64.77" y1="63.5" x2="53.34" y2="63.5" width="0.1524" layer="91"/>
-<label x="53.34" y="63.5" size="1.778" layer="95"/>
-</segment>
-<segment>
 <label x="68.58" y="-63.5" size="1.778" layer="95" rot="R180"/>
 <pinref part="Q5" gate="G$1" pin="G"/>
 <wire x1="68.58" y1="-63.5" x2="33.02" y2="-63.5" width="0.1524" layer="91"/>
 </segment>
+<segment>
+<pinref part="JL1" gate="G$1" pin="P$2"/>
+<wire x1="64.77" y1="50.8" x2="53.34" y2="50.8" width="0.1524" layer="91"/>
+<label x="53.34" y="50.8" size="1.778" layer="95"/>
+</segment>
 </net>
 <net name="SV1" class="0">
-<segment>
-<pinref part="JL1" gate="G$1" pin="P$10"/>
-<wire x1="64.77" y1="60.96" x2="53.34" y2="60.96" width="0.1524" layer="91"/>
-<label x="53.34" y="60.96" size="1.778" layer="95"/>
-</segment>
 <segment>
 <label x="68.58" y="-50.8" size="1.778" layer="95" rot="R180"/>
@@
 <wire x1="68.58" y1="-50.8" x2="33.02" y2="-50.8" width="0.1524" layer="91"/>
 </segment>
-</net>
+<segment>
+<pinref part="JL1" gate="G$1" pin="P$4"/>
+<wire x1="64.77" y1="53.34" x2="53.34" y2="53.34" width="0.1524" layer="91"/>
+<label x="53.34" y="53.34" size="1.778" layer="95"/>
+</segment>
+</net>

Commit message: Add files via upload
Changed lines of the file:
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@@
 <instance part="U1" gate="G$1" x="96.52" y="15.24"/>
 <instance part="JL1" gate="G$1" x="71.12" y="58.42"/>
-<instance part="SVETLA" gate="A" x="-12.7" y="-12.7"/>
+<instance part="SVETLA" gate="A" x="-12.7" y="-12.7" smashed="yes">
+<attribute name="NAME" x="-19.05" y="-4.445" size="1.778" layer="95"/>
+<attribute name="VALUE" x="-19.05" y="-20.32" size="1.778" layer="96"/>
+</instance>
 <instance part="Q3" gate="G$1" x="30.48" y="-38.1" rot="MR270"/>
-<instance part="Q1" gate="G$1" x="30.48" y="-25.4" rot="MR270"/>
+<instance part="Q1" gate="G$1" x="30.48" y="-25.4" smashed="yes" rot="MR270">
+<attribute name="NAME" x="29.845" y="-30.48" size="1.27" layer="95" rot="MR270"/>
+<attribute name="VALUE" x="31.75" y="-30.48" size="1.27" layer="96" rot="MR270"/>
+</instance>
 <instance part="Q4" gate="G$1" x="30.48" y="-53.34" rot="MR270"/>
 <instance part="Q5" gate="G$1" x="30.48" y="-66.04" rot="MR270"/>
