File: Columba2/car2r0.sch (EAGLE design)
At the start: 65 parts, among them J2 DS1014-14S, Q1 16MHz, U2 WT8266, U3 FT231XS

Commit message: VCU V5 WIP 2
Parts:
- added C14, C15, C16: 100nF, rcl:C-EUC1206
- added R-SMI: (no value), resistor:R-TRIMM5W
- added R23: 10k, custom:R-EU_R0603
- added RS1, RS2: 0.1R (CS06FTFUR100), custom:R-EU_R1206
- added X1: JST-XH-04-PIN-LONG-PAD, Rembrandt Electronics - JST XH Connectors v1-0:JST-XH-04-PIN-LONG-PAD
- renumbered STRJ1 to MS1, STRJ2 to MS2, U$1 to SDRV
Connections:
- net N$8 renamed VREG
- removed net ENABLEN: SDRV.ENABLEN
- removed net N$4: GPIO.3, MCU.(A14)PC6
- removed net RESETN: SDRV.!RESET
- removed net SLEEPN: SDRV.!SLEEP
- new net CP1: C14.1, SDRV.CP1
- new net CP2: C14.2, SDRV.CP2
- new net N$8: GPIO.4, MCU.(A14)PC6
- new net OUT1A: SDRV.OUT1A, X1-2.S
- new net OUT1B: SDRV.OUT1B, X1-1.S
- new net OUT2A: SDRV.OUT2A, X1-3.S
- new net OUT2B: SDRV.OUT2B, X1-4.S
- new net SENSE1: RS2.1, SDRV.SENSE1
- new net SENSE2: RS1.1, SDRV.SENSE2
- new net SIV: R-SMI.A, R23.1
- new net STEP_EN: MCU.(AD3)PA3, SDRV.ENABLEN
- new net STEP_RST: MCU.(AD1)PA1, SDRV.!RESET
- new net STEP_SLEEP: MCU.(AD2)PA2, SDRV.!SLEEP
- new net SVREF: C16.1, R-SMI.S, SDRV.REF
- new net VCP: C15.1, SDRV.VCP
- net 5V: now also C15.2, R23.2, SDRV.VBB1, SDRV.VBB2
- net DIR: now also MCU.(AD4)PA4
- net GND: now also C16.2, R-SMI.E, RS1.2, RS2.2, SDRV.GND
- net N$3: now also GPIO.3; no longer GPIO.4
- net STEP: now also MCU.(OC3B/INT4)PE4
Other:
- note added: "Stepper Max Current Trimmer"
- moved on the sheet: C11, Q3
