File: Columba2/car2r0.brd (EAGLE design)
At the start: 55 x 58 mm, 65 parts, among them J2 DS1014-14S, Q1 16MHz, U2 WT8266, U3 FT231XS

Commit message: VCU V5 WIP 2
Parts:
- removed STRJ1, STRJ2: (no value), pinhead:1X02
- removed U$1: A4982LP, columba:TSSOP24P
- added C14, C15, C16: 100nF, rcl:C1206
- added MS1, MS2: (no value), pinhead:1X02
- added R-SMI: (no value), resistor:RTRIM5W
- added R23: 10k, custom:R0603
- added RS1, RS2: 0.1R (CS06FTFUR100), custom:R1206
- added SDRV: A4982LP, columba:TSSOP24P
- added X1: JST-XH-04-PIN-LONG-PAD, Rembrandt Electronics - JST XH Connectors v1-0:JST-XH-04-PACKAGE-LONG-PAD
- moved C11 87.7 mm to (47.7, 53.4), turned to 90 degrees
- moved J2 27.7 mm to (31.4, 54.4), turned to 180 degrees
- moved Q3 14.5 mm to (28.4, 47.6)
- moved SPKR 14.5 mm to (34.1, 48.5)
- moved GPIO 4.30 mm to (44.0, 23.2), turned to 180 degrees
Connections:
- removed net ENABLEN: U$1.23
- removed net N$4: GPIO.3, MCU.59
- removed net RESETN: U$1.7
- removed net SLEEPN: U$1.9
- new net CP1: C14.1, SDRV.1
- new net CP2: C14.2, SDRV.2
- new net OUT1A: SDRV.18, X1.2
- new net OUT1B: SDRV.15, X1.1
- new net OUT2A: SDRV.19, X1.3
- new net OUT2B: SDRV.22, X1.4
- new net SENSE1: RS2.1, SDRV.17
- new net SENSE2: RS1.1, SDRV.20
- new net SIV: R-SMI.1, R23.1
- new net STEP_EN: MCU.75, SDRV.23
- new net STEP_RST: MCU.77, SDRV.7
- new net STEP_SLEEP: MCU.76, SDRV.9
- new net SVREF: C16.1, R-SMI.2, SDRV.12
- new net VCP: C15.1, SDRV.3
- new net VREG: C11.1, SDRV.4
- net 5V: now also C15.2, MS1.1, MS2.2, R23.2, SDRV.10, SDRV.16, SDRV.21, SDRV.8; no longer STRJ1.1, STRJ2.2, U$1.10, U$1.8
- net DIR: now also MCU.74, SDRV.14; no longer U$1.14
- net GND: now also C16.2, R-SMI.3, RS1.2, RS2.2, SDRV.13, SDRV.24, SDRV.PAD; no longer U$1.13, U$1.24, U$1.PAD
- net MS1: now also MS1.2, SDRV.5; no longer STRJ1.2, U$1.5
- net MS2: now also MS2.1, SDRV.6; no longer STRJ2.1, U$1.6
- net N$3: now also GPIO.3; no longer GPIO.4
- net N$8: now also GPIO.4, MCU.59; no longer C11.1, U$1.4
- net STEP: now also MCU.6, SDRV.11; no longer U$1.11
Routing:
- net 5V: track 215.0 -> 268.7 mm, vias 7 -> 12
- net GND: track 242.3 -> 195.2 mm, vias 8 -> 6
- net OUT2A: track 0.00 -> 29.9 mm
- net OUT1A: track 0.00 -> 29.6 mm
- net STEP: track 0.00 -> 29.6 mm, vias 0 -> 2
- net BSM_A: track 22.0 -> 0.00 mm, vias 1 -> 0
- net PX_EN: track 21.0 -> 0.00 mm, vias 2 -> 0
- net STEP_RST: track 0.00 -> 20.9 mm, vias 0 -> 2
- net PX4: track 19.4 -> 0.00 mm, vias 1 -> 0
- net OUT2B: track 0.00 -> 18.5 mm
- net OUT1B: track 0.00 -> 18.4 mm
- net PX3: track 17.2 -> 0.00 mm, vias 1 -> 0
- net STEP_EN: track 0.00 -> 16.9 mm, vias 0 -> 2
- net STEP_SLEEP: track 0.00 -> 16.8 mm, vias 0 -> 2
- net SPKR: track 16.6 -> 0.00 mm, vias 2 -> 0
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Other:
- board text removed: "ON"

Commit message: VCU V5.0 (Final)
Parts:
- moved Q3 7.76 mm to (35.6, 44.7)
- moved PWRLED 4.40 mm to (9.10, 6.30)
- moved R20 4.12 mm to (9.10, 9.10)
- moved SPKR 1.63 mm to (35.8, 48.2)
- moved C15 0.14 mm to (50.5, 50.2), turned to 115 degrees
Routing:
- net VIN: track 64.5 -> 9.93 mm
- net 5V: track 268.7 -> 301.2 mm, vias 12 -> 13
- net SPM_PWM: track 25.2 -> 0.00 mm, vias 1 -> 0
- net BSA1: track 0.00 -> 18.9 mm, vias 0 -> 1
- net PX_EN: track 0.00 -> 18.7 mm
- net BSA0: track 0.00 -> 18.2 mm, vias 0 -> 1
- net LX0: track 0.00 -> 17.2 mm
- net BSM_A: track 0.00 -> 16.3 mm, vias 0 -> 1
- net BSM_B: track 0.00 -> 15.6 mm, vias 0 -> 1
- net BSM_C: track 0.00 -> 14.9 mm, vias 0 -> 3
- net LX3: track 3.25 -> 17.5 mm, vias 0 -> 1
- net BSAI: track 0.00 -> 14.1 mm, vias 0 -> 1
- net LX2: track 3.00 -> 16.9 mm, vias 0 -> 1
- net LX1: track 2.75 -> 16.4 mm, vias 0 -> 1
- net MOSI: track 19.7 -> 12.8 mm
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Other:
- board text added: "Columba"
- board text added: "VCU V5 Rev. 0"
- board text added: "VCU V5.0"
- board text removed: "VCU V4 Rev. 1"
